Commit message: URDF: Alle Achsen korrekt und Paketnamen gefixt

File: src/hand_description/urdf/urdf.xacro (robot description, xacro)
@@ -3,8 +3,9 @@
      Commit Version: 1.6.0-4-g7f85cfe  Build Version: 1.6.7995.38578
      For more information, please see http://wiki.ros.org/sw_urdf_exporter -->
-<robot
-  name="bionic_hand">
+  <robot
+    name="bionic_hand">
+    <!-- World Link als neuer Root -->
   <link name="world"/>
-    <!-- Joint um die Hand richtig zu orientieren -->
+  <!-- Joint um die Hand richtig zu orientieren -->
   <joint name="world_to_base" type="fixed">
     <parent link="world"/>
@@ -16,15 +17,15 @@
     <inertial>
       <origin
-        xyz="0.03958 -0.029691 0.015244"
-        rpy="0 0 0" />
-      <mass
-        value="0.65238" />
-      <inertia
-        ixx="0.00082112"
-        ixy="8.9286E-05"
-        ixz="3.3707E-05"
-        iyy="0.0014836"
-        iyz="-1.6843E-05"
-        izz="0.0010714" />
+        xyz="0.03912886852115 -0.02936264886893 0.0154057797768061"
+        rpy="0 0 0" />
+      <mass
+        value="0.648187431870064" />
+      <inertia
+        ixx="0.000817855553979597"
+        ixy="8.875849584592E-05"
+        ixz="3.31929662839044E-05"
+        iyy="0.00148537892208656"
+        iyz="-1.75158796634625E-05"
+        izz="0.00106984032112581" />
     </inertial>
     <visual>
@@ -39,5 +40,5 @@
         name="">
         <color
-          rgba="0.79216 0.81961 0.93333 1" />
+          rgba="0.792156862745098 0.819607843137255 0.933333333333333 1" />
       </material>
     </visual>
@@ -53,40 +54,40 @@
   </link>
   <link
-    name="thumb">
-    <inertial>
-      <origin
-        xyz="-0.0310468955754792 0.0146728189340897 -0.01641634870464"
-        rpy="0 0 0" />
-      <mass
-        value="0.0188289535395376" />
-      <inertia
-        ixx="4.4591837920961E-06"
-        ixy="-5.53558786935455E-07"
-        ixz="1.37851662185635E-06"
-        iyy="6.98550535645012E-06"
-        iyz="6.4443900077485E-07"
-        izz="6.12233605411629E-06" />
-    </inertial>
-    <visual>
-      <origin
-        xyz="0 0 0"
-        rpy="0 0 0" />
-      <geometry>
-        <mesh
-          filename="package://hand_description/meshes/thumb.STL" />
-      </geometry>
-      <material
-        name="">
-        <color
-          rgba="0.792156862745098 0.819607843137255 0.933333333333333 1" />
-      </material>
-    </visual>
-    <collision>
-      <origin
-        xyz="0 0 0"
-        rpy="0 0 0" />
-      <geometry>
-        <mesh
-          filename="package://hand_description/meshes/thumb.STL" />
+    name="thumb_opposition">
+    <inertial>
+      <origin
+        xyz="-0.030921850566624 0.0146727324061557 -0.0164392665314555"
+        rpy="0 0 0" />
+      <mass
+        value="0.0188289789775585" />
+      <inertia
+        ixx="4.45919280552344E-06"
+        ixy="-5.53559993158624E-07"
+        ixz="1.37851508545918E-06"
+        iyy="6.98551165055523E-06"
+        iyz="6.4444143928376E-07"
+        izz="6.12234363761581E-06" />
+    </inertial>
+    <visual>
+      <origin
+        xyz="0 0 0"
+        rpy="0 0 0" />
+      <geometry>
+        <mesh
+          filename="package://hand_description/meshes/thumb_opposition.STL" />
+      </geometry>
+      <material
+        name="">
+        <color
+          rgba="0.792156862745098 0.819607843137255 0.933333333333333 1" />
+      </material>
+    </visual>
+    <collision>
+      <origin
+        xyz="0 0 0"
+        rpy="0 0 0" />
+      <geometry>
+        <mesh
+          filename="package://hand_description/meshes/thumb_opposition.STL" />
       </geometry>
     </collision>
@@ -96,13 +97,14 @@
     type="revolute">
     <origin
-      xyz="-0.044432 -0.029203 0.0043878"
-      rpy="1.987 0.073988 0.015374" />
+      xyz="-0.044557 -0.029225 0.0043879"
+      rpy="1.1887 -0.068156 0.01342" />
     <parent
       link="base_link" />
     <child
-      link="thumb" />
+      link="thumb_opposition" />
     <axis
       xyz="0.98363 -0.0005966 -0.18021" />
-    <limit lower="-1.57" upper="1.57" effort="10" velocity="1"/>
+    <limit
+      lower="-1.57" upper="1.57" effort="10" velocity="1"/>
   </joint>
   <link
@@ -110,15 +112,15 @@
     <inertial>
       <origin
-        xyz="0.00752395524320154 0.00186096944336717 -0.00320605716681524"
-        rpy="0 0 0" />
-      <mass
-        value="0.00899609220397239" />
-      <inertia
-        ixx="7.08057279665508E-07"
-        ixy="1.356946672071E-07"
-        ixz="-2.45328917532297E-07"
-        iyy="1.18390467499842E-06"
-        iyz="1.18726954796414E-07"
-        izz="1.06737478504705E-06" />
+        xyz="0.00485254318295213 0.0115774656855361 -0.0178189490794952"
+        rpy="0 0 0" />
+      <mass
+        value="0.00899608808051006" />
+      <inertia
+        ixx="7.08057425667585E-07"
+        ixy="1.35694118393264E-07"
+        ixz="-2.45328865431087E-07"
+        iyy="1.18390389757121E-06"
+        iyz="1.18726868091096E-07"
+        izz="1.06737398415733E-06" />
     </inertial>
     <visual>
@@ -150,13 +152,14 @@
     type="revolute">
     <origin
-      xyz="-0.031243 0.027955 -0.036949"
-      rpy="0 0 0" />
-    <parent
-      link="thumb" />
+      xyz="-0.028446 0.018239 -0.022359"
+      rpy="-0.047586 0.12392 -0.19596" />
+    <parent
+      link="thumb_opposition" />
     <child
       link="thumb_rotation" />
     <axis
       xyz="0.1505 -0.54739 0.82323" />
-    <limit lower="-1.57" upper="1.57" effort="10" velocity="1"/>
+    <limit
+      lower="-1.57" upper="1.57" effort="10" velocity="1"/>
   </joint>
   <link
@@ -164,15 +167,15 @@
     <inertial>
       <origin
-        xyz="-0.0155706619077729 0.00107314934487866 0.00626879225058935"
-        rpy="0 0 0" />
-      <mass
-        value="0.00685717177436016" />
-      <inertia
-        ixx="3.11754853031797E-07"
-        ixy="9.27034426999804E-08"
-        ixz="6.38349131015559E-08"
-        iyy="1.08304711854349E-06"
-        iyz="-5.41424395732265E-09"
-        izz="1.32280787234435E-06" />
+        xyz="-0.0155706608829484 0.00107315483017915 0.0062687915604831"
+        rpy="0 0 0" />
+      <mass
+        value="0.00685716829419009" />
+      <inertia
+        ixx="3.11754832187612E-07"
+        ixy="9.27036628856027E-08"
+        ixz="6.38349944365018E-08"
+        iyy="1.08304708866608E-06"
+        iyz="-5.41431302860761E-09"
+        izz="1.32280779786269E-06" />
     </inertial>
     <visual>
@@ -204,6 +207,6 @@
     type="revolute">
     <origin
-      xyz="0.00073166 0.0086002 -0.012265"
-      rpy="2.3445 -0.40101 -0.39979" />
+      xyz="-0.0019397 0.018317 -0.026878"
+      rpy="2.1608 0.12026 0.016692" />
     <parent
       link="thumb_rotation" />
@@ -212,5 +215,6 @@
     <axis
       xyz="0.17549 -0.00010644 0.98448" />
-    <limit lower="-1.57" upper="1.57" effort="10" velocity="1"/>
+    <limit
+      lower="-1.57" upper="1.57" effort="10" velocity="1"/>
   </joint>
   <link
@@ -218,15 +222,15 @@
     <inertial>
       <origin
-        xyz="-0.034785521476525 -0.0200301266994405 -0.0109240437666255"
-        rpy="0 0 0" />
-      <mass
-        value="0.00215756775239621" />
-      <inertia
-        ixx="5.47658702851547E-08"
-        ixy="1.88954857927782E-08"
-        ixz="3.69651145948474E-08"
-        iyy="2.22364902291839E-07"
-        iyz="-3.41420293869522E-09"
-        izz="2.52589614872599E-07" />
+        xyz="-0.00718053252045824 0.000724409234434703 -0.00147454565081055"
+        rpy="0 0 0" />
+      <mass
+        value="0.00215756681963284" />
+      <inertia
+        ixx="5.47658542119838E-08"
+        ixy="1.88954712154763E-08"
+        ixz="3.69651100914208E-08"
+        iyy="2.22364898192174E-07"
+        iyz="-3.41419343155599E-09"
+        izz="2.52589616879644E-07" />
     </inertial>
     <visual>
@@ -258,6 +262,6 @@
     type="revolute">
     <origin
-      xyz="0.0024822 0 0.013925"
-      rpy="-0.12191 -0.047997 -0.75062" />
+      xyz="-0.032276 0.0026768 0.0057535"
+      rpy="0.017774 -0.00089913 0.099874" />
     <parent
       link="thumb_mcp_flexion" />
@@ -266,5 +270,6 @@
     <axis
       xyz="0.17549 -0.00010644 0.98448" />
-    <limit lower="-1.57" upper="1.57" effort="10" velocity="1"/>
+    <limit
+      lower="-1.57" upper="1.57" effort="10" velocity="1"/>
   </joint>
   <link
@@ -272,15 +277,15 @@
     <inertial>
       <origin
-        xyz="-0.0568441579315472 -0.0299741007495122 -0.0115227782932227"
-        rpy="0 0 0" />
-      <mass
-        value="0.00422716702426551" />
-      <inertia
-        ixx="1.40124491068462E-07"
-        ixy="5.49789778918847E-09"
-        ixz="9.16911669230519E-09"
-        iyy="2.42390316052478E-07"
-        iyz="-1.42163523160784E-08"
-        izz="2.1985487203313E-07" />
+        xyz="-0.00701799183672533 -0.00401755261035154 0.0040895075655876"
+        rpy="0 0 0" />
+      <mass
+        value="0.00422718056224681" />
+      <inertia
+        ixx="1.40125013203282E-07"
+        ixy="5.49842510113702E-09"
+        ixz="9.16944340087911E-09"
+        iyy="2.42391220941455E-07"
+        iyz="-1.42164042694292E-08"
+        izz="2.19856077912689E-07" />
     </inertial>
     <visual>
@@ -312,6 +317,6 @@
     type="revolute">
     <origin
-      xyz="0.0017489 0 0.0098114"
-      rpy="-0.028947 -0.0023481 -0.16308" />
+      xyz="-0.024063 0.0027904 0.0042895"
+      rpy="-0.00063934 0 -0.0035867" />
     <parent
       link="thumb_pip" />
@@ -320,5 +325,6 @@
     <axis
       xyz="0.17549 -0.00010644 0.98448" />
-    <limit lower="-1.57" upper="1.57" effort="10" velocity="1"/>
+    <limit
+      lower="-1.57" upper="1.57" effort="10" velocity="1"/>
   </joint>
   <link
@@ -326,15 +332,15 @@
     <inertial>
       <origin
-        xyz="-0.000909500913099874 0.0190949489863932 0.00491034741633578"
-        rpy="0 0 0" />
-      <mass
-        value="0.00962736795097376" />
-      <inertia
-        ixx="3.02657286197391E-06"
-        ixy="3.09347950580268E-08"
-        ixz="-6.74461457482812E-08"
-        iyy="1.66118262653521E-06"
-        iyz="-4.11078346082898E-08"
-        izz="1.78273306499507E-06" />
+        xyz="-0.000909442206088804 0.0190949661941328 0.00490966953133031"
+        rpy="0 0 0" />
+      <mass
+        value="0.00962689371201742" />
+      <inertia
+        ixx="3.02649913257995E-06"
+        ixy="3.09387520209351E-08"
+        ixz="-6.74558178094872E-08"
+        iyy="1.661110752292E-06"
+        iyz="-4.11033806607042E-08"
+        izz="1.78272744485798E-06" />
     </inertial>
     <visual>
@@ -367,5 +373,5 @@
     <origin
       xyz="-0.12274 -0.01291 0.0017357"
-      rpy="0.072567 -0.15899 1.3249" />
+      rpy="0.0040501 -0.1746 1.7321" />
     <parent
       link="base_link" />
@@ -374,59 +380,61 @@
     <axis
       xyz="0 0 1" />
-    <limit lower="-1.57" upper="1.57" effort="10" velocity="1"/>
-  </joint>
-  <link
-    name="mcp_flexion">
-    <inertial>
-      <origin
-        xyz="-0.0533173021213905 0.0147626054460368 0.0129986079628866"
-        rpy="0 0 0" />
-      <mass
-        value="0.00685716892835977" />
-      <inertia
-        ixx="3.11754907458993E-07"
-        ixy="9.27036913286524E-08"
-        ixz="6.3835062205085E-08"
-        iyy="1.08304734782688E-06"
-        iyz="-5.41431208162088E-09"
-        izz="1.32280813298493E-06" />
-    </inertial>
-    <visual>
-      <origin
-        xyz="0 0 0"
-        rpy="0 0 0" />
-      <geometry>
-        <mesh
-          filename="package://hand_description/meshes/mcp_flexion.STL" />
-      </geometry>
-      <material
-        name="">
-        <color
-          rgba="0.792156862745098 0.819607843137255 0.933333333333333 1" />
-      </material>
-    </visual>
-    <collision>
-      <origin
-        xyz="0 0 0"
-        rpy="0 0 0" />
-      <geometry>
-        <mesh
-          filename="package://hand_description/meshes/mcp_flexion.STL" />
-      </geometry>
-    </collision>
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
Commit message: Feierabend-Push: Optimierte Servo-Steuerung mit 100Hz
- DynamixelSDK Integration mit 4Mbps Baudrate
- Neuer servo_mapper_node mit 100Hz Timer
- Optimierte Frequenz-Synchronisation (28Hz → 100Hz)
- Deadband-Filter für stabile Servo-Kommunikation
- .gitignore für DynamixelSDK und SCServo
- Launch-Datei für komplette Hand-Steuerung
- URDF mit Mimic-Joints für DIP-Gelenke

Performance: 100Hz stabile Servo-Steuerung erreicht!

File: src/hand_description/urdf/urdf.xacro (robot description, xacro)
@@ -327,4 +327,5 @@
     <limit
       lower="-1.57" upper="1.57" effort="10" velocity="1"/>
+    <mimic joint="thumb_pip" multiplier="0.9"/>
   </joint>
   <link
@@ -447,10 +448,10 @@
         value="0.0021575700735159" />
       <inertia
-        ixx="5.47658929498861E-08"
+        ixx="5.47658542119838E-08"
         ixy="1.88954712154763E-08"
-        ixz="3.69651213830989E-08"
-        iyy="2.22364898660454E-07"
+        ixz="3.69651100914208E-08"
+        iyy="2.22364898192174E-07"
         iyz="-3.41421563770417E-09"
-        izz="2.52589630171238E-07" />
+        izz="2.52589616879644E-07" />
     </inertial>
     <visual>
@@ -547,4 +548,5 @@
     <limit
       lower="-1.57" upper="1.57" effort="10" velocity="1"/>
+    <mimic joint="index_pip" multiplier="0.9"/>
   </joint>
   <link
@@ -654,5 +656,5 @@
       link="middle_mcp_flexion" />
     <axis
-      xyz="-0.17549 0.00010644 -0.98448" />
+      xyz="0.17549 -0.00010644 0.98448" />
     <limit
       lower="-1.57" upper="1.57" effort="10" velocity="1"/>
@@ -669,5 +671,5 @@
         ixx="5.4765889602427E-08"
         ixy="1.8895496022229E-08"
-        ixz="3.69651226560766E-08"
+        ixz="3.69651213830989E-08"
         iyy="2.22364893977912E-07"
         iyz="-3.41420959985044E-09"
@@ -709,5 +711,5 @@
       link="middle_pip" />
     <axis
-      xyz="-0.17549 0.00010644 -0.98448" />
+      xyz="0.17549 -0.00010644 0.98448" />
     <limit
       lower="-1.57" upper="1.57" effort="10" velocity="1"/>
@@ -767,4 +769,5 @@
     <limit
       lower="-1.57" upper="1.57" effort="10" velocity="1"/>
+    <mimic joint="middle_pip" multiplier="0.9"/>
   </joint>
   <link
@@ -946,5 +949,5 @@
         ixz="9.16976614596534E-09"
         iyy="2.42392426432486E-07"
-        iyz="-1.42164439566301E-08"
+        iyz="-1.42164042694292E-08"
         izz="2.19857467650712E-07" />
     </inertial>
@@ -987,4 +990,5 @@
     <limit
       lower="-1.57" upper="1.57" effort="10" velocity="1"/>
+    <mimic joint="ring_pip" multiplier="0.9"/>
   </joint>
 </robot>
